File: hardware/panel/main.kicad_pcb (KiCad board)
At the start: 2 copper layers, 80 x 80 mm, 54 parts, among them J1 LOAD_CON, J2 Conn_01x08, J3 SD_CARD, J4 ENCODER, SW1 CC, SW2 CV, SW3 CR, SW4 CP, SW5 EN, U1 ESP32-DEVKIT-V1

Commit message: hardware: panel: Small pins and plane adjustments
* Adjusted pins for sockets to be bigger
* Regenerated gnp plane
Routing:
- net GND: track 376.2 -> 377.3 mm
- net +5V: track 136.7 -> 137.6 mm
- net /DISPLAY/CS: track 44.7 -> 44.1 mm
