File: hardware/load/supplies.kicad_sch (KiCad schematic)
At the start: 14 parts, among them U601 L7812, U602 L7805, U603 LM1117MP-3.3

Commit message: feat(load): fix DRC errors and warinigs
Parts:
- JP601, JP602, JP603, JP604: footprint Jumper:SolderJumper-2_P1.3mm_Open_TrianglePad1.0x1.5mm -> Load:SolderJumper-2_P1.3mm_Open_TrianglePad1.0x1.5mm
Changed lines of the file:
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@@
 			)
 		)
-		(property "Footprint" "Jumper:SolderJumper-2_P1.3mm_Open_TrianglePad1.0x1.5mm"
+		(property "Footprint" "Load:SolderJumper-2_P1.3mm_Open_TrianglePad1.0x1.5mm"
 			(at 50.8 64.77 0)
 			(effects
@@
 			)
 		)
-		(property "Footprint" "Jumper:SolderJumper-2_P1.3mm_Open_TrianglePad1.0x1.5mm"
+		(property "Footprint" "Load:SolderJumper-2_P1.3mm_Open_TrianglePad1.0x1.5mm"
 			(at 156.21 64.77 0)
 			(effects
@@
 			)
 		)
-		(property "Footprint" "Jumper:SolderJumper-2_P1.3mm_Open_TrianglePad1.0x1.5mm"
+		(property "Footprint" "Load:SolderJumper-2_P1.3mm_Open_TrianglePad1.0x1.5mm"
 			(at 107.95 64.77 0)
 			(effects
@@
 			)
 		)
-		(property "Footprint" "Jumper:SolderJumper-2_P1.3mm_Open_TrianglePad1.0x1.5mm"
+		(property "Footprint" "Load:SolderJumper-2_P1.3mm_Open_TrianglePad1.0x1.5mm"
 			(at 212.09 64.77 0)
 			(effects
