File: hardware/load/driver.kicad_sch (KiCad schematic)
At the start: 18 parts, among them Q302 2sb1357, U301 LM324

Commit message: feat(load): route logic and optmize layout
Parts:
- removed JP301: enable_analog_feedback, Jumper:SolderJumper-3_P2.0mm_Open_TrianglePad1.0x1.5mm, symbol Jumper:Jumper_3_Open
Connections:
- net at U301.8: now also C302.2, C303.2, R304.1
Changed lines of the file:
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@@
+	)
+	(junction
+		(at 100.33 121.92)
+		(diameter 0)
+		(color 0 0 0 0)
+	)
+	(junction
+		(at 173.99 119.38)
+		(diameter 0)
+		(color 0 0 0 0)
+	)
+	(junction
+		(at 135.89 137.16)
+		(diameter 0)
+		(color 0 0 0 0)
+	)
+	(junction
+		(at 198.12 116.84)
+		(diameter 0)
+		(color 0 0 0 0)
 	)
 	(junction
@@
 	)
 	(junction
-		(at 100.33 121.92)
-		(diameter 0)
-		(color 0 0 0 0)
-	)
-	(junction
-		(at 173.99 119.38)
-		(diameter 0)
-		(color 0 0 0 0)
-	)
-	(junction
-		(at 135.89 137.16)
-		(diameter 0)
-		(color 0 0 0 0)
-	)
-	(junction
-		(at 198.12 116.84)
-		(diameter 0)
-		(color 0 0 0 0)
-	)
-	(junction
 		(at 92.71 121.92)
-		(diameter 0)
-		(color 0 0 0 0)
-	)
-	(junction
-		(at 100.33 116.84)
 		(diameter 0)
 		(color 0 0 0 0)
@@
 	(wire
 		(pts
-			(xy 142.24 115.57) (xy 142.24 99.06)
-		)
-		(stroke
-			(width 0)
-			(type default)
-		)
-	)
-	(wire
-		(pts
 			(xy 234.95 121.92) (xy 234.95 132.08)
 		)
@@
 	(wire
 		(pts
+			(xy 135.89 137.16) (xy 135.89 119.38)
+		)
+		(stroke
+			(width 0)
+			(type default)
+		)
+	)
+	(wire
+		(pts
+			(xy 92.71 121.92) (xy 92.71 137.16)
+		)
+		(stroke
+			(width 0)
+			(type default)
+		)
+	)
+	(wire
+		(pts
+			(xy 86.36 116.84) (xy 106.68 116.84)
+		)
+		(stroke
+			(width 0)
+			(type default)
+		)
+	)
+	(wire
+		(pts
+			(xy 162.56 102.87) (xy 162.56 105.41)
+		)
+		(stroke
+			(width 0)
+			(type default)
+		)
+	)
+	(wire
+		(pts
+			(xy 234.95 77.47) (xy 234.95 80.01)
+		)
+		(stroke
+			(width 0)
+			(type default)
+		)
+	)
+	(wire
+		(pts
+			(xy 86.36 121.92) (xy 92.71 121.92)
+		)
+		(stroke
+			(width 0)
+			(type default)
+		)
+	)
+	(wire
+		(pts
+			(xy 234.95 148.59) (xy 236.22 148.59)
+		)
+		(stroke
+			(width 0)
+			(type default)
+		)
+	)
+	(wire
+		(pts
 			(xy 135.89 119.38) (xy 161.29 119.38)
 		)
@@
 	(wire
 		(pts
-			(xy 135.89 137.16) (xy 135.89 119.38)
-		)
-		(stroke
-			(width 0)
-			(type default)
-		)
-	)
-	(wire
-		(pts
-			(xy 92.71 121.92) (xy 92.71 137.16)
-		)
-		(stroke
-			(width 0)
-			(type default)
-		)
-	)
-	(wire
-		(pts
-			(xy 86.36 116.84) (xy 100.33 116.84)
-		)
-		(stroke
-			(width 0)
-			(type default)
-		)
-	)
-	(wire
-		(pts
-			(xy 162.56 102.87) (xy 162.56 105.41)
-		)
-		(stroke
-			(width 0)
-			(type default)
-		)
-	)
-	(wire
-		(pts
-			(xy 234.95 77.47) (xy 234.95 80.01)
-		)
-		(stroke
-			(width 0)
-			(type default)
-		)
-	)
-	(wire
-		(pts
-			(xy 86.36 121.92) (xy 92.71 121.92)
-		)
-		(stroke
-			(width 0)
-			(type default)
-		)
-	)
-	(wire
-		(pts
-			(xy 234.95 148.59) (xy 236.22 148.59)
-		)
-		(stroke
-			(width 0)
-			(type default)
-		)
-	)
-	(wire
-		(pts
-			(xy 129.54 115.57) (xy 127 115.57)
-		)
-		(stroke
-			(width 0)
-			(type default)
-		)
-	)
-	(wire
-		(pts
 			(xy 118.11 149.86) (xy 135.89 149.86)
 		)
@@
 	(wire
 		(pts
-			(xy 100.33 99.06) (xy 100.33 116.84)
-		)
-		(stroke
-			(width 0)
-			(type default)
-		)
-	)
-	(wire
-		(pts
 			(xy 166.37 99.06) (xy 173.99 99.06)
 		)
@@
 	(wire
 		(pts
-			(xy 121.92 119.38) (xy 127 119.38)
-		)
-		(stroke
-			(width 0)
-			(type default)
-		)
-	)
-	(wire
-		(pts
-			(xy 142.24 99.06) (xy 100.33 99.06)
+			(xy 121.92 119.38) (xy 135.89 119.38)
 		)
 		(stroke
@@
 	(wire
 		(pts
-			(xy 100.33 116.84) (xy 106.68 116.84)
-		)
-		(stroke
-			(width 0)
-			(type default)
-		)
-	)
-	(wire
-		(pts
 			(xy 173.99 132.08) (xy 173.99 119.38)
 		)
@@
 		(pts
 			(xy 110.49 137.16) (xy 125.73 137.16)
-		)
-		(stroke
-			(width 0)
-			(type default)
-		)
-	)
-	(wire
-		(pts
-			(xy 127 115.57) (xy 127 119.38)
 		)
 		(stroke
@@
 					(unit 1)
 				)
-			)
-		)
-	)
-	(symbol
-		(lib_id "Jumper:Jumper_3_Open")
-		(at 135.89 115.57 0)
-		(unit 1)
-		(exclude_from_sim yes)
-		(in_bom no)
-		(on_board yes)
-		(dnp no)
-		(fields_autoplaced yes)
-		(property "Reference" "JP301"
-			(at 135.89 109.22 0)
-			(effects
-				(font
-					(size 1.27 1.27)
-				)
-			)
-		)
-		(property "Value" "enable_analog_feedback"
-			(at 135.89 111.76 0)
-			(effects
-				(font
-					(size 1.27 1.27)
-				)
-			)
-		)
-		(property "Footprint" "Jumper:SolderJumper-3_P2.0mm_Open_TrianglePad1.0x1.5mm"
-			(at 135.89 115.57 0)
-			(effects
-				(font
-					(size 1.27 1.27)
-				)
-				(hide yes)
-			)
-		)
-		(property "Datasheet" "~"
-			(at 135.89 115.57 0)
-			(effects
-				(font
-					(size 1.27 1.27)
-				)
-				(hide yes)
-			)
-		)
-		(property "Description" "Jumper, 3-pole, both open"
-			(at 135.89 115.57 0)
-			(effects
-				(font
-					(size 1.27 1.27)
-				)
-				(hide yes)
-			)
-		)
-		(pin "3"
-		)
-		(pin "2"
-		)
-		(pin "1"
-		)
-		(instances
-			(project "main"
-				(path "/03550a2d-ebcf-48cb-96c1-fbf16f6a9151/c796216b-1ecc-4454-aec0-b824777ffdda"
-					(reference "JP301")
-					(unit 1)
-				)

Commit message: feat(load): modify analog PID values on the schematic
Parts:
- C301: value C_Small -> 100n
- C302: value C_Small -> NC
- C303: value C_Small -> 10n
- R301: value 3k3 -> 2k7
- R302: value 3k3 -> 250R
- R303: value 3k3 -> 330
Changed lines of the file:
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@@
 			)
 		)
-		(property "Value" "3k3"
+		(property "Value" "250R"
 			(at 83.82 124.46 90)
 			(effects
@@
 			)
 		)
-		(property "Value" "C_Small"
+		(property "Value" "NC"
 			(at 115.5763 153.67 90)
 			(effects
@@
 			)
 		)
-		(property "Value" "3k3"
+		(property "Value" "330"
 			(at 107.95 139.7 90)
 			(effects
@@
 			)
 		)
-		(property "Value" "3k3"
+		(property "Value" "2k7"
 			(at 74.93 139.7 90)
 			(effects
@@
 			)
 		)
-		(property "Value" "C_Small"
+		(property "Value" "10n"
 			(at 128.2763 140.97 90)
 			(effects
@@
 			)
 		)
-		(property "Value" "C_Small"
+		(property "Value" "100n"
 			(at 67.3163 125.73 90)
 			(effects
