File: hardware/load/stm32.kicad_sch (KiCad schematic)
At the start: 9 parts, among them U201 BluePill

Commit message: feat(load): route logic and optmize layout
Parts:
- added D203, D204: 3.3 < V < 5.1, Diode_SMD:D_MiniMELF, symbol Device:D_Zener
- added R203, R204: 2.2k, Resistor_SMD:R_0805_2012Metric_Pad1.20x1.40mm_HandSolder, symbol Device:R_Small
Connections:
- net GND: now also D203.2 (A), D204.2 (A)
- net adc_alert: now also U201.34 (PB1); no longer U201.13 (PB5)
- net fan: now also U201.5 (PA8); no longer U201.31 (PA6)
- net at R202.1: now also U201.33 (PB0); no longer U201.34 (PB1)
- net at U201.22 (PC13): now also D203.1 (K), R204.2
- net at U201.23 (PC14): now also D204.1 (K), R203.2
- net at U201.32 (PA7): now also R201.1
- new net external_trigger_in: R203.1
- new net external_trigger_out: R204.1
- no-connect marks 23 -> 18
Other:
- moved on the sheet: D201, D202, R201, R202

Commit message: feat(load): fix DRC errors and warinigs
Parts:
- JP201, JP202: footprint Jumper:SolderJumper-2_P1.3mm_Open_TrianglePad1.0x1.5mm -> Load:SolderJumper-2_P1.3mm_Open_TrianglePad1.0x1.5mm
Changed lines of the file:
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@@
 			)
 		)
-		(property "Footprint" "Jumper:SolderJumper-2_P1.3mm_Open_TrianglePad1.0x1.5mm"
+		(property "Footprint" "Load:SolderJumper-2_P1.3mm_Open_TrianglePad1.0x1.5mm"
 			(at 38.1 26.67 0)
 			(effects
@@
 			)
 		)
-		(property "Footprint" "Jumper:SolderJumper-2_P1.3mm_Open_TrianglePad1.0x1.5mm"
+		(property "Footprint" "Load:SolderJumper-2_P1.3mm_Open_TrianglePad1.0x1.5mm"
 			(at 38.1 33.02 0)
 			(effects

Commit message: feat(load): modify analog PID values on the schematic
Connections:
- net enable_load: now reaches U201.13 (PB5)
Changed lines of the file:
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@@
+	(wire
+		(pts
+			(xy 93.98 134.62) (xy 102.87 134.62)
+		)
+		(stroke
+			(width 0)
+			(type default)
+		)
+	)
 	(wire
 		(pts
@@
 		)
 	)
+	(hierarchical_label "enable_load"
+		(shape input)
+		(at 93.98 134.62 180)
+		(fields_autoplaced yes)
+		(effects
+			(font
+				(size 1.27 1.27)
+			)
+			(justify right)
+		)
+	)
