File: hardware/hmi/display.kicad_sch (KiCad schematic)
At the start: 8 parts, among them J2 Conn_01x08

Commit message: fix: conect DC pin and change reset to avoid conflicts with UART
Connections:
- net DC: now reaches J2.6 (Pin_6)
- no-connect marks 1 -> 0
Changed lines of the file:
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@@
 		(color 0 0 0 0)
 	)
-	(no_connect
-		(at 135.89 85.09)
-	)
 	(wire
 		(pts
@@
 	(wire
 		(pts
+			(xy 134.62 85.09) (xy 135.89 85.09)
+		)
+		(stroke
+			(width 0)
+			(type default)
+		)
+	)
+	(wire
+		(pts
 			(xy 123.19 95.25) (xy 123.19 100.33)
 		)
@@
 		(fields_autoplaced yes)
 		(effects
+			(font
+				(size 1.27 1.27)
+			)
+			(justify right)
+		)
+	)
+	(hierarchical_label "DC"
+		(shape input)
+		(at 134.62 85.09 180)
+		(fields_autoplaced yes)
+		(effects
