File: hardware/hmi/main.kicad_sch (KiCad schematic)
At the start: 5 parts, among them J1 LOAD_CON

Commit message: fix: conect DC pin and change reset to avoid conflicts with UART
Other:
- sheet DISPLAY ports: added DC; removed none
- sheet ESP32 ports: added LCD_DC; removed none
Changed lines of the file:
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@@
+	(wire
+		(pts
+			(xy 137.16 130.81) (xy 138.43 130.81)
+		)
+		(stroke
+			(width 0)
+			(type default)
+		)
+	)
 	(wire
 		(pts
@@
 	(wire
 		(pts
+			(xy 138.43 153.67) (xy 151.13 153.67)
+		)
+		(stroke
+			(width 0)
+			(type default)
+		)
+	)
+	(wire
+		(pts
 			(xy 140.97 128.27) (xy 137.16 128.27)
 		)
@@
 		(pts
 			(xy 80.01 50.8) (xy 83.82 50.8)
+		)
+		(stroke
+			(width 0)
+			(type default)
+		)
+	)
+	(wire
+		(pts
+			(xy 138.43 130.81) (xy 138.43 153.67)
 		)
 		(stroke
@@
 	(sheet
 		(at 114.3 80.01)
-		(size 22.86 50.8)
+		(size 22.86 53.34)
 		(fields_autoplaced yes)
 		(stroke
@@
 		)
 		(property "Sheetfile" "esp32.kicad_sch"
-			(at 114.3 131.3946 0)
+			(at 114.3 133.9346 0)
 			(effects
 				(font
@@
 		(pin "BTN_CC" input
 			(at 137.16 82.55 0)
+			(effects
+				(font
+					(size 1.27 1.27)
+				)
+				(justify right)
+			)
+		)
+		(pin "LCD_DC" input
+			(at 137.16 130.81 0)
 			(effects
 				(font
@@
 	(sheet
 		(at 151.13 134.62)
-		(size 12.7 19.05)
+		(size 12.7 22.86)
 		(fields_autoplaced yes)
 		(stroke
@@
 		)
 		(property "Sheetfile" "display.kicad_sch"
-			(at 151.13 154.2546 0)
+			(at 151.13 158.0646 0)
 			(effects
 				(font
@@
 			(effects
 				(font
+					(size 1.27 1.27)
+				)
+				(justify left)
+			)
+		)
+		(pin "DC" input
+			(at 151.13 153.67 180)
+			(effects
+				(font
