File: hardware/hmi/esp32.kicad_sch (KiCad schematic)
At the start: 6 parts, among them U1 ESP32-DEVKIT-V1

Commit message: WIP hardware
Connections:
- net SCL: now also U1.12 (GPIO_3/RX0)
- net SDA: now also U1.13 (GPIO_1/TX0)
- no-connect marks 9 -> 7
Changed lines of the file:
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@@
+	)
+	(junction
+		(at 165.1 99.06)
+		(diameter 0)
+		(color 0 0 0 0)
 	)
 	(junction
@@
 	)
 	(junction
+		(at 162.56 96.52)
+		(diameter 0)
+		(color 0 0 0 0)
+	)
+	(junction
 		(at 116.84 66.04)
 		(diameter 0)
@@
 	)
 	(no_connect
-		(at 158.75 109.22)
-	)
-	(no_connect
 		(at 105.41 113.03)
 	)
@@
 		(at 105.41 130.81)
 	)
-	(no_connect
-		(at 158.75 111.76)
-	)
 	(wire
 		(pts
@@
 	(wire
 		(pts
+			(xy 165.1 111.76) (xy 165.1 99.06)
+		)
+		(stroke
+			(width 0)
+			(type default)
+		)
+	)
+	(wire
+		(pts
 			(xy 130.81 66.04) (xy 130.81 78.74)
 		)
@@
 	(wire
 		(pts
+			(xy 162.56 109.22) (xy 162.56 96.52)
+		)
+		(stroke
+			(width 0)
+			(type default)
+		)
+	)
+	(wire
+		(pts
 			(xy 161.29 88.9) (xy 166.37 88.9)
 		)
@@
 	(wire
 		(pts
-			(xy 166.37 96.52) (xy 161.29 96.52)
+			(xy 166.37 96.52) (xy 162.56 96.52)
 		)
 		(stroke
@@
 	(wire
 		(pts
+			(xy 162.56 96.52) (xy 161.29 96.52)
+		)
+		(stroke
+			(width 0)
+			(type default)
+		)
+	)
+	(wire
+		(pts
 			(xy 133.35 138.43) (xy 134.62 138.43)
 		)
@@
 	(wire
 		(pts
+			(xy 158.75 111.76) (xy 165.1 111.76)
+		)
+		(stroke
+			(width 0)
+			(type default)
+		)
+	)
+	(wire
+		(pts
 			(xy 110.49 66.04) (xy 116.84 66.04)
 		)
@@
 	(wire
 		(pts
+			(xy 165.1 99.06) (xy 161.29 99.06)
+		)
+		(stroke
+			(width 0)
+			(type default)
+		)
+	)
+	(wire
+		(pts
 			(xy 158.75 118.11) (xy 166.37 118.11)
 		)
@@
 	(wire
 		(pts
-			(xy 166.37 99.06) (xy 161.29 99.06)
+			(xy 166.37 99.06) (xy 165.1 99.06)
 		)
 		(stroke
@@
 		)
 		(stroke
+			(width 0)
+			(type default)
+		)
+	)
+	(wire
+		(pts
+			(xy 158.75 109.22) (xy 162.56 109.22)
+		)
+		(stroke
