File: hardware/hmi/esp32.kicad_sch (KiCad schematic)
At the start: 6 parts, among them U1 ESP32-DEVKIT-V1

Commit message: fix: conect DC pin and change reset to avoid conflicts with UART
Connections:
- net LCD_RST: now also U1.6 (GPIO_16/RX2); no longer U1.12 (GPIO_3/RX0)
- net LCD_DC: now reaches U1.3 (GPIO_15_/ADC_13)
Changed lines of the file:
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@@
-	)
-	(no_connect
-		(at 158.75 120.65)
 	)
 	(no_connect
@@
 		(at 105.41 130.81)
 	)
+	(no_connect
+		(at 158.75 111.76)
+	)
 	(wire
 		(pts
@@
 	(wire
 		(pts
+			(xy 158.75 130.81) (xy 165.1 130.81)
+		)
+		(stroke
+			(width 0)
+			(type default)
+		)
+	)
+	(wire
+		(pts
 			(xy 132.08 137.16) (xy 132.08 138.43)
 		)
@@
 	(wire
 		(pts
-			(xy 158.75 111.76) (xy 166.37 111.76)
+			(xy 158.75 120.65) (xy 166.37 120.65)
 		)
 		(stroke
@@
 	(hierarchical_label "LCD_RST"
 		(shape input)
-		(at 166.37 111.76 0)
+		(at 166.37 120.65 0)
 		(fields_autoplaced yes)
 		(effects
@@
 		(fields_autoplaced yes)
 		(effects
+			(font
+				(size 1.27 1.27)
+			)
+			(justify left)
+		)
+	)
+	(hierarchical_label "LCD_DC"
+		(shape input)
+		(at 165.1 130.81 0)
+		(fields_autoplaced yes)
+		(effects

Commit message: hardware: hmi: Change to UART
Connections:
- net SCL: now also U1.12 (GPIO_3/RX0)
- net SDA: now also U1.13 (GPIO_1/TX0)
- no-connect marks 9 -> 7
Changed lines of the file:
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@@
-	)
-	(no_connect
-		(at 158.75 109.22)
 	)
 	(no_connect
@@
 		(at 105.41 130.81)
 	)
-	(no_connect
-		(at 158.75 111.76)
-	)
 	(wire
 		(pts
@@
 	(wire
 		(pts
+			(xy 158.75 111.76) (xy 166.37 111.76)
+		)
+		(stroke
+			(width 0)
+			(type default)
+		)
+	)
+	(wire
+		(pts
 			(xy 110.49 72.39) (xy 110.49 73.66)
 		)
@@
 	(wire
 		(pts
+			(xy 158.75 109.22) (xy 166.37 109.22)
+		)
+		(stroke
+			(width 0)
+			(type default)
+		)
+	)
+	(wire
+		(pts
 			(xy 110.49 67.31) (xy 110.49 66.04)
 		)
@@
 		)
 	)
+	(hierarchical_label "SCL"
+		(shape input)
+		(at 166.37 111.76 0)
+		(fields_autoplaced yes)
+		(effects
+			(font
+				(size 1.27 1.27)
+			)
+			(justify left)
+		)
+	)
 	(hierarchical_label "MISO"
 		(shape input)
@@
 		(fields_autoplaced yes)
 		(effects
+			(font
+				(size 1.27 1.27)
+			)
+			(justify left)
+		)
+	)
+	(hierarchical_label "SDA"
+		(shape input)
+		(at 166.37 109.22 0)
+		(fields_autoplaced yes)
+		(effects
